File: PCB/EPD/EPD.kicad_pcb (KiCad board)
At the start: 4 copper layers, 70 x 70 mm, 67 parts, among them J1 Conn_01x26, J2 Shelly, J3 USB-PROG, J4 BTN2, J6 BTN2, J7 USB-C-Socket-V, J8 PWR, P1 +, P10 2, P11 2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

Commit message: Update
Parts:
- C17, C18: value 4.7uF -> 4.7uF 50V; footprint RevK:C_0402 -> RevK:C_0805
- L1: value 10uH -> 470uH
- L2: value 10uH -> 47uH 1.3A
- moved J7 1.39 mm to (108.2, 102.8)
- moved C17 1.04 mm to (108.1, 75.5)
- moved L1 0.32 mm to (110.7, 84.4)
Routing:
- net Net-(J7-CC1): track 14.5 -> 18.4 mm
- net GND: track 30.8 -> 34.6 mm, vias 24 -> 17
- net Net-(D3-A): track 19.8 -> 18.6 mm
- net PWR: track 19.9 -> 18.8 mm
- net +3.3V: track 84.4 -> 83.5 mm
- net Net-(J1-Pin_24): track 9.83 -> 9.31 mm
Other:
- copper layers 4 -> 2
