File: PCB/EPD/EPD.kicad_sch (KiCad schematic)
At the start: 69 parts, among them J1 Conn_01x26, J2 Shelly, J3 USB-PROG, J4 BTN2, J6 BTN2, J7 USB-C-Socket-V, J8 PWR, P1 +, P10 2, P11 2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

Commit message: Update
Parts:
- C17, C18: value 4.7uF -> 4.7uF 50V; footprint RevK:C_0402 -> RevK:C_0805
- L1: value 10uH -> 470uH; MPN (none) -> C42429207
- L2: value 10uH -> 47uH 1.3A; MPN (none) -> C602032

Commit message: Library update
Parts:
- L2: value 47uH 1.3A -> 10uH; MPN C602032 -> C42428017
Changed lines of the file:
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@@
 			)
 		)
-		(property "Value" "47uH 1.3A"
+		(property "Value" "10uH"
 			(at 191.77 45.72 90)
 			(effects
@@
 			)
 		)
-		(property "MPN" "C602032"
+		(property "MPN" "C42428017"
 			(at 185.42 45.72 90)
 			(effects
