File: PCB/EPD75NFC/EPD75.kicad_sch (KiCad schematic)
At the start: 172 parts, among them J1 Conn_01x26, J10 TF_PUSH, J11 Reset, J12 TC2030-USB-NL-DS, J2 PWR, J3 NFC, J4 BTN, J5 USB-C-Socket-H, J6 TEMP, J7 USB-C-Socket-H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

Commit message: Library update
Parts:
- added C127, C82: 220uF Tant, RevK:CP_EIA-3528-21_Kemet-B, symbol Device:C_Polarized
- added J9: OUT, RevK:WAGO-2060-452-998-404, symbol Connector_Generic:Conn_01x02
- added U6, U8, U9: TPS22916CNYFPR, RevK:WCSP-4-0.78x0.78, symbol RevK:TPS22916
- C28: value C_Polarized -> 220uF Tant; footprint RevK:CP_EIA-7343-31_Kemet-D -> RevK:CP_EIA-3528-21_Kemet-B; MPN C106188 -> C122649
- U3: MPN C3659294 -> C3659362
Connections:
- net +3.3V: now also C127.1, U6.A2 (VIN), U9.A2 (VIN); no longer C11.1, C18.2, C67.1, C68.2, C69.2, C70.2, J1.15 (Pin_15), J1.16 (Pin_16), JP1.3 (B), L1.2
- net GND: now also C127.2, C82.2, J9.1 (Pin_1), U6.B1 (GND), U8.B1 (GND), U9.B1 (GND)
- net NFC5V: now also U8.A1 (VOUT); no longer J2.2 (Pin_2)
- net PEPD: now reaches U4.15 (GPIO11)
- net PEPD: now also U9.B2 (ON)
- net PNFC: now reaches U4.16 (GPIO12)
- net PNFC: now also U8.B2 (ON)
- net POUT: now reaches U4.17 (GPIO13)
- net POUT: now also U6.B2 (ON)
- new net: J9.2 (Pin_2), U6.A1 (VOUT)
- new net EPD3V3: C11.1, C18.2, C67.1, C68.2, C69.2, C70.2, J1.15 (Pin_15), J1.16 (Pin_16), JP1.3 (B), L1.2, U9.A1 (VOUT)
- new net NFCIN: C82.1, J2.2 (Pin_2), U8.A2 (VIN)
- no-connect marks 35 -> 32
